Commit message: xacro modified to reference local mesh directory

File: nuturtle_description/urdf/turtlebot3_burger.urdf.xacro (robot description, xacro)
@@ -1,6 +1,6 @@
 <?xml version="1.0" ?>
 <robot name="turtlebot3_burger" xmlns:xacro="http://ros.org/wiki/xacro">
-  <xacro:include filename="$(find turtlebot3_description)/urdf/common_properties.xacro"/>
-  <xacro:include filename="$(find turtlebot3_description)/urdf/turtlebot3_burger.gazebo.xacro"/>
+  <xacro:include filename="$(find nuturtle_description)/urdf/common_properties.xacro"/>
+  <xacro:include filename="$(find nuturtle_description)/urdf/turtlebot3_burger.gazebo.xacro"/>
   <link name="base_footprint"/>
   <joint name="base_joint" type="fixed">
@@ -13,5 +13,5 @@
       <origin xyz="-0.032 0 0.0" rpy="0 0 0"/>
       <geometry>
-        <mesh filename="package://turtlebot3_description/meshes/bases/burger_base.stl" scale="0.001 0.001 0.001"/>
+        <mesh filename="package://nuturtle_description/meshes/burger_base.stl" scale="0.001 0.001 0.001"/>
       </geometry>
       <material name="light_black"/>
@@ -41,5 +41,5 @@
       <origin xyz="0 0 0" rpy="1.57 0 0"/>
       <geometry>
-        <mesh filename="package://turtlebot3_description/meshes/wheels/left_tire.stl" scale="0.001 0.001 0.001"/>
+        <mesh filename="package://nuturtle_description/meshes/left_tire.stl" scale="0.001 0.001 0.001"/>
       </geometry>
       <material name="dark"/>
@@ -69,5 +69,5 @@
       <origin xyz="0 0 0" rpy="1.57 0 0"/>
       <geometry>
-        <mesh filename="package://turtlebot3_description/meshes/wheels/right_tire.stl" scale="0.001 0.001 0.001"/>
+        <mesh filename="package://nuturtle_description/meshes/right_tire.stl" scale="0.001 0.001 0.001"/>
       </geometry>
       <material name="dark"/>
@@ -122,5 +122,5 @@
       <origin xyz="0 0 0.0" rpy="0 0 0"/>
       <geometry>
-        <mesh filename="package://turtlebot3_description/meshes/sensors/lds.stl" scale="0.001 0.001 0.001"/>
+        <mesh filename="package://turtlebot3_description/meshes/lds.stl" scale="0.001 0.001 0.001"/>
       </geometry>
       <material name="dark"/>

Commit message: finished A.2. Need to figure out and remove 3rd xacro/urdf file at some point.

File: nuturtle_description/urdf/turtlebot3_burger.urdf.xacro (robot description, xacro)
@@ -122,5 +122,5 @@
       <origin xyz="0 0 0.0" rpy="0 0 0"/>
       <geometry>
-        <mesh filename="package://turtlebot3_description/meshes/lds.stl" scale="0.001 0.001 0.001"/>
+        <mesh filename="package://nuturtle_description/meshes/lds.stl" scale="0.001 0.001 0.001"/>
       </geometry>
       <material name="dark"/>

Commit message: Task A.3 completed

File: nuturtle_description/urdf/turtlebot3_burger.urdf.xacro (robot description, xacro)
@@ -3,4 +3,8 @@
   <xacro:include filename="$(find nuturtle_description)/urdf/common_properties.xacro"/>
   <xacro:include filename="$(find nuturtle_description)/urdf/turtlebot3_burger.gazebo.xacro"/>
+  <xacro:property name="diff_params" value="$(find nuturtle_description)/config/diff_params.yaml"/>
+  <xacro:property name="drive" value="${load_yaml(diff_params)}"/>
+  <xacro:property name="wheel_radius" value="${drive['wheel_radius']}"/>
+  <xacro:property name="track_width" value="${drive['track_width']}"/>
   <link name="base_footprint"/>
   <joint name="base_joint" type="fixed">
@@ -34,5 +38,5 @@
     <parent link="base_link"/>
     <child link="wheel_left_link"/>
-    <origin xyz="0.0 0.08 0.023" rpy="-1.57 0 0"/>
+    <origin xyz="0.0 ${0.5*track_width} 0.023" rpy="-1.57 0 0"/>
     <axis xyz="0 0 1"/>
   </joint>
@@ -48,5 +52,5 @@
       <origin xyz="0 0 0" rpy="0 0 0"/>
       <geometry>
-        <cylinder length="0.018" radius="0.033"/>
+        <cylinder length="0.018" radius="${wheel_radius}"/>
       </geometry>
     </collision>
@@ -62,5 +66,5 @@
     <parent link="base_link"/>
     <child link="wheel_right_link"/>
-    <origin xyz="0.0 -0.080 0.023" rpy="-1.57 0 0"/>
+    <origin xyz="0.0 ${-0.5*track_width} 0.023" rpy="-1.57 0 0"/>
     <axis xyz="0 0 1"/>
   </joint>
@@ -76,5 +80,5 @@
       <origin xyz="0 0 0" rpy="0 0 0"/>
       <geometry>
-        <cylinder length="0.018" radius="0.033"/>
+        <cylinder length="0.018" radius="${wheel_radius}"/>
       </geometry>
     </collision>

Commit message: first attempt at making color argument

File: nuturtle_description/urdf/turtlebot3_burger.urdf.xacro (robot description, xacro)
@@ -19,5 +19,7 @@
         <mesh filename="package://nuturtle_description/meshes/burger_base.stl" scale="0.001 0.001 0.001"/>
       </geometry>
-      <material name="light_black"/>
+      <!-- This is what we need to change the color of  -->
+      <!-- <material name="light_black"/> -->
+      <material name="$(arg color)"/>
     </visual>
     <collision>

Commit message: cleaned up fixed frames in rviz

File: nuturtle_description/urdf/turtlebot3_burger.urdf.xacro (robot description, xacro)
@@ -7,11 +7,11 @@
   <xacro:property name="wheel_radius" value="${drive['wheel_radius']}"/>
   <xacro:property name="track_width" value="${drive['track_width']}"/>
-  <link name="base_footprint"/>
-  <joint name="base_joint" type="fixed">
-    <parent link="base_footprint"/>
-    <child link="base_link"/>
+  <link name="$(arg color)-base_footprint"/>
+  <joint name="$(arg color)-base_joint" type="fixed">
+    <parent link="$(arg color)-base_footprint"/>
+    <child link="$(arg color)-base_link"/>
     <origin xyz="0.0 0.0 0.010" rpy="0 0 0"/>
   </joint>
-  <link name="base_link">
+  <link name="$(arg color)-base_link">
     <visual>
       <origin xyz="-0.032 0 0.0" rpy="0 0 0"/>
@@ -38,5 +38,5 @@
   </link>
   <joint name="wheel_left_joint" type="continuous">
-    <parent link="base_link"/>
+    <parent link="$(arg color)-base_link"/>
     <child link="wheel_left_link"/>
     <origin xyz="0.0 ${0.5*track_width} 0.023" rpy="-1.57 0 0"/>
@@ -66,5 +66,5 @@
   </link>
   <joint name="wheel_right_joint" type="continuous">
-    <parent link="base_link"/>
+    <parent link="$(arg color)-base_link"/>
     <child link="wheel_right_link"/>
     <origin xyz="0.0 ${-0.5*track_width} 0.023" rpy="-1.57 0 0"/>
@@ -94,5 +94,5 @@
   </link>
   <joint name="caster_back_joint" type="fixed">
-    <parent link="base_link"/>
+    <parent link="$(arg color)-base_link"/>
     <child link="caster_back_link"/>
     <origin xyz="-0.081 0 -0.004" rpy="-1.57 0 0"/>
@@ -114,5 +114,5 @@
   </link>
   <joint name="imu_joint" type="fixed">
-    <parent link="base_link"/>
+    <parent link="$(arg color)-base_link"/>
     <child link="imu_link"/>
     <origin xyz="-0.032 0 0.068" rpy="0 0 0"/>
@@ -120,5 +120,5 @@
   <link name="imu_link"/>
   <joint name="scan_joint" type="fixed">
-    <parent link="base_link"/>
+    <parent link="$(arg color)-base_link"/>
     <child link="base_scan"/>
     <origin xyz="-0.032 0 0.172" rpy="0 0 0"/>

Commit message: multiple robots now showing up in one rviz window

File: nuturtle_description/urdf/turtlebot3_burger.urdf.xacro (robot description, xacro)
@@ -4,5 +4,5 @@
   <xacro:include filename="$(find nuturtle_description)/urdf/turtlebot3_burger.gazebo.xacro"/>
   <xacro:property name="diff_params" value="$(find nuturtle_description)/config/diff_params.yaml"/>
-  <xacro:property name="drive" value="${load_yaml(diff_params)}"/>
+  <xacro:property name="drive" value="${xacro.load_yaml(diff_params)}"/>
   <xacro:property name="wheel_radius" value="${drive['wheel_radius']}"/>
   <xacro:property name="track_width" value="${drive['track_width']}"/>

Commit message: made some changes robot's visible in rviz now

File: nuturtle_description/urdf/turtlebot3_burger.urdf.xacro (robot description, xacro)
@@ -37,11 +37,11 @@
     </inertial>
   </link>
-  <joint name="wheel_left_joint" type="continuous">
+  <joint name="$(arg color)-wheel_left_joint" type="continuous">
     <parent link="$(arg color)-base_link"/>
-    <child link="wheel_left_link"/>
+    <child link="$(arg color)-wheel_left_link"/>
     <origin xyz="0.0 ${0.5*track_width} 0.023" rpy="-1.57 0 0"/>
     <axis xyz="0 0 1"/>
   </joint>
-  <link name="wheel_left_link">
+  <link name="$(arg color)-wheel_left_link">
     <visual>
       <origin xyz="0 0 0" rpy="1.57 0 0"/>
@@ -65,11 +65,11 @@
       </inertial>
   </link>
-  <joint name="wheel_right_joint" type="continuous">
+  <joint name="$(arg color)-wheel_right_joint" type="continuous">
     <parent link="$(arg color)-base_link"/>
-    <child link="wheel_right_link"/>
+    <child link="$(arg color)-wheel_right_link"/>
     <origin xyz="0.0 ${-0.5*track_width} 0.023" rpy="-1.57 0 0"/>
     <axis xyz="0 0 1"/>
   </joint>
-  <link name="wheel_right_link">
+  <link name="$(arg color)-wheel_right_link">
     <visual>
       <origin xyz="0 0 0" rpy="1.57 0 0"/>
@@ -93,10 +93,10 @@
       </inertial>
   </link>
-  <joint name="caster_back_joint" type="fixed">
+  <joint name="$(arg color)-caster_back_joint" type="fixed">
     <parent link="$(arg color)-base_link"/>
-    <child link="caster_back_link"/>
+    <child link="$(arg color)-caster_back_link"/>
     <origin xyz="-0.081 0 -0.004" rpy="-1.57 0 0"/>
   </joint>
-  <link name="caster_back_link">
+  <link name="$(arg color)-caster_back_link">
     <collision>
       <origin xyz="0 0.001 0" rpy="0 0 0"/>

Commit message: finished A.7

File: nuturtle_description/urdf/turtlebot3_burger.urdf.xacro (robot description, xacro)
@@ -6,4 +6,5 @@
   <xacro:property name="wheel_radius" value="${drive['wheel_radius']}"/>
   <xacro:property name="track_width" value="${drive['track_width']}"/>
+  <xacro:property name="collision_radius" value="${drive['collision_radius']}"/>
   <link name="$(arg color)-base_footprint"/>
   <joint name="$(arg color)-base_joint" type="fixed">
@@ -25,5 +26,10 @@
       <origin xyz="-0.032 0 0.070" rpy="0 0 0"/>
       <geometry>
-        <box size="0.140 0.140 0.143"/>
+        <xacro:if value="${collision_radius > 0.0}">
+          <cylinder radius="${collision_radius}" length="0.143"/>
+        </xacro:if>
+        <xacro:if value="${collision_radius == 0.0}">
+          <box size="0.140 0.140 0.143"/>
+        </xacro:if>
       </geometry>
     </collision>

Commit message: noise and markers tentatively work correctly

File: nuturtle_description/urdf/turtlebot3_burger.urdf.xacro (robot description, xacro)
@@ -126,8 +126,8 @@
   <joint name="scan_joint" type="fixed">
     <parent link="$(arg color)-base_link"/>
-    <child link="base_scan"/>
+    <child link="$(arg color)-base_scan"/>
     <origin xyz="-0.032 0 0.172" rpy="0 0 0"/>
   </joint>
-  <link name="base_scan">
+  <link name="$(arg color)-base_scan">
     <visual>
       <origin xyz="0 0 0.0" rpy="0 0 0"/>
